Commit message: article publish

File: jackal_description/urdf/accessories.urdf.xacro (robot description, xacro)
@@ -13,432 +13,118 @@
   <!-- This optional plate mounts both the upgraded GPS and the Velodyne 3D LIDAR. -->
   <xacro:include filename="$(find jackal_description)/urdf/accessories/bridge_plate.urdf.xacro" />
-  <!-- 2D Lidars -->
-  <xacro:include filename="$(find sick_tim)/urdf/sick_tim.urdf.xacro" />
-  <xacro:include filename="$(find lms1xx)/urdf/sick_lms1xx.urdf.xacro" />
-  <xacro:include filename="$(find jackal_description)/urdf/accessories/sick_lms1xx_inverted_mount.urdf.xacro" />
-  <xacro:include filename="$(find jackal_description)/urdf/accessories/sick_lms1xx_upright_mount.urdf.xacro" />
-  <xacro:include filename="$(find jackal_description)/urdf/accessories/hokuyo_utm30.urdf.xacro" />
-  <xacro:include filename="$(find jackal_description)/urdf/accessories/hokuyo_ust10.urdf.xacro" />
-  <xacro:include filename="$(find jackal_description)/urdf/accessories/vlp16_mount.urdf.xacro" />
-  <xacro:include filename="$(find jackal_description)/urdf/accessories/hdl32_mount.urdf.xacro" />
-  <!--
-    Add Microstrain IMU. By default the Jackal comes equipped with an IMU linked to "imu_link". These extra
-    optional microstrain IMU's will be added to another frame, by default, "microstrain_link".
-  -->
-  <xacro:if value="$(optenv JACKAL_IMU_MICROSTRAIN 0)">
-    <xacro:property name="frame"  value="$(optenv JACKAL_IMU_MICROSTRAIN_LINK microstrain_link)"/>
-    <xacro:property name="parent" value="$(optenv JACKAL_IMU_MICROSTRAIN_PARENT base_link)"/>
-    <xacro:property name="xyz"    value="$(optenv JACKAL_IMU_MICROSTRAIN_OFFSET -0.139 0.096 0.100)"/>
-    <xacro:property name="rpy"    value="$(optenv JACKAL_IMU_MICROSTRAIN_RPY ${PI} 0 -${PI/2})"/>
-    <link name="${frame}" />
-    <joint name="${frame}_joint" type="fixed">
-      <parent link="${parent}" />
-      <child link="${frame}" />
-      <origin xyz="${xyz}" rpy="${rpy}" />
+  <!-- If enabled, generate the LASER payload (by default, a SICK LMS111). -->
+  <xacro:if value="$(optenv JACKAL_LASER 0)">
+    <xacro:if value="$(optenv JACKAL_LASER_HOKUYO 0)">
+      <xacro:include filename="$(find jackal_description)/urdf/accessories/hokuyo_ust10.urdf.xacro" />
+      <hokuyo_ust10_mount prefix="$(optenv JACKAL_LASER_MOUNT front)"
+                          parent_link="$(optenv JACKAL_LASER_MOUNT front)_mount"
+                          topic="$(optenv JACKAL_LASER_TOPIC front/scan)" />
+    </xacro:if>
+    <xacro:unless value="$(optenv JACKAL_LASER_HOKUYO 0)">
+      <xacro:include filename="$(find jackal_description)/urdf/accessories/sick_lms1xx_mount.urdf.xacro" />
+      <sick_lms1xx_mount prefix="$(optenv JACKAL_LASER_MOUNT front)"
+                         parent_link="$(optenv JACKAL_LASER_MOUNT front)_mount"
+                         topic="$(optenv JACKAL_LASER_TOPIC front/scan)"/>
+    </xacro:unless>
+  </xacro:if>
+  <!-- If enabled, generate the upgraded Navsat payload (a Novatel Smart6). -->
+  <xacro:if value="$(optenv JACKAL_NAVSAT 0)">
+    <xacro:include filename="$(find jackal_description)/urdf/accessories/novatel_smart6.urdf.xacro" />
+    <bridge_plate mount="$(optenv JACKAL_NAVSAT_MOUNT rear)"
+                  height="$(optenv JACKAL_NAVSAT_HEIGHT 0.1)" />
+    <novatel_smart6 prefix="$(optenv JACKAL_NAVSAT_MOUNT rear)"/>
+    <joint name="$(optenv JACKAL_NAVSAT_MOUNT rear)_navsat_joint" type="fixed">
+      <origin xyz="0 0 0" rpy="0 0 0" />
+      <parent link="$(optenv JACKAL_NAVSAT_MOUNT rear)_bridge" />
+      <child link="$(optenv JACKAL_NAVSAT_MOUNT rear)_navsat" />
     </joint>
   </xacro:if>
-  <!--
-    Add primary/secondary 2D lidar sensors.  By default these are SICK LMS1xx but can be changed with the
-    JACKAL_LASER_MODEL and JACKAL_LASER_SECONDARY_MODEL environment variables. Valid model designations are:
-    - lms1xx (default) :: SICK LMS1xx
-    - ust10            :: Hokuyo UST10
-    - utm30            :: Hokuyo UTM30
-  -->
-  <!-- Primary 2D Lidar -->
-  <xacro:if value="$(optenv JACKAL_LASER 0)">
-    <xacro:property name="mount" value="$(optenv JACKAL_LASER_MOUNT front)" />
-    <xacro:property name="topic" value="$(optenv JACKAL_LASER_TOPIC front/scan)" />
-    <xacro:property name="tower" value="$(optenv JACKAL_LASER_TOWER 1)" />
-    <xacro:property name="prefix" value="$(optenv JACKAL_LASER_PREFIX ${mount})" />
-    <xacro:property name="parent" value="$(optenv JACKAL_LASER_PARENT ${mount}_mount)" />
-    <xacro:property name="lidar_model" value="$(optenv JACKAL_LASER_MODEL lms1xx)" />
-    <xacro:property name="mount_type" value="$(optenv JACKAL_LASER_MOUNT_TYPE upright)" />
-    <!-- SICK LMS1xx -->
-    <xacro:if value="${lidar_model == 'lms1xx'}">
-      <!-- Mount Enabled -->
-      <xacro:if value="${tower}">
-        <xacro:if value="${mount_type == 'upright'}">
-          <xacro:sick_lms1xx_upright_mount topic="${topic}" prefix="${prefix}" parent_link="${parent}">
-            <origin xyz="$(optenv JACKAL_LASER_OFFSET 0 0 0)" rpy="$(optenv JACKAL_LASER_RPY 0 0 0)" />
-          </xacro:sick_lms1xx_upright_mount>
-        </xacro:if>
-        <xacro:if value="${mount_type == 'inverted'}">
-          <xacro:sick_lms1xx_inverted_mount topic="${topic}" prefix="${prefix}" parent_link="${parent}">
-            <origin xyz="$(optenv JACKAL_LASER_OFFSET 0 0 0)" rpy="$(optenv JACKAL_LASER_RPY 0 0 0)" />
-          </xacro:sick_lms1xx_inverted_mount>
-        </xacro:if>
-      </xacro:if>
-      <!-- Mount Disabled -->
-      <xacro:unless value="${tower}">
-        <xacro:sick_lms1xx frame="${prefix}_laser" topic="${topic}" />
-        <link name="${prefix}_laser_base"/>
-        <joint name="${prefix}_laser_base_joint" type="fixed">
-          <origin xyz="$(optenv JACKAL_LASER_OFFSET 0 0 0)" rpy="$(optenv JACKAL_LASER_RPY 0 0 0)"/>
-          <parent link="${parent}"/>
-          <child link="${prefix}_laser_base"/>
-        </joint>
-        <joint name="${prefix}_laser_joint" type="fixed">
-          <origin xyz="0 0 0.116" rpy="0 0 0"/>
-          <parent link="${prefix}_laser_base"/>
-          <child link="${prefix}_laser"/>
-        </joint>
-      </xacro:unless>
-    </xacro:if>
-    <!-- SICK Tim -->
-    <xacro:if value="${lidar_model == 'tim551'}">
-      <xacro:property name="prefix" value="$(optenv JACKAL_LASER_PREFIX tim551)" />
-      <xacro:sick_tim551 name="${prefix}" ros_topic="${topic}"/>
-      <joint name="${prefix}_mount_link_joint" type="fixed">
-        <origin xyz="$(optenv JACKAL_LASER_OFFSET 0 0 0)" rpy="$(optenv JACKAL_LASER_RPY 0 0 0)"/>
-        <parent link="${parent}"/>
-        <child link="${prefix}_mount_link"/>
-      </joint>
-    </xacro:if>
-    <!-- Hokuyo UST10 -->
-    <xacro:if value="${lidar_model == 'ust10'}">
-      <xacro:hokuyo_ust10_mount topic="${topic}" prefix="${prefix}" parent_link="${parent}">
-        <origin xyz="$(optenv JACKAL_LASER_OFFSET 0 0 0)" rpy="$(optenv JACKAL_LASER_RPY 0 0 0)" />
-      </xacro:hokuyo_ust10_mount>
-    </xacro:if>
-    <!-- Hokuyo UTM30 -->
-    <xacro:if value="${lidar_model == 'utm30'}">
-      <xacro:hokuyo_utm30_mount topic="${topic}" prefix="${prefix}" parent_link="${parent}">
-        <origin xyz="$(optenv JACKAL_LASER_OFFSET 0 0 0)" rpy="$(optenv JACKAL_LASER_RPY 0 0 0)" />
-      </xacro:hokuyo_utm30_mount>
-    </xacro:if>
-  </xacro:if>
-  <!-- Secondary 2D Lidar -->
-  <xacro:if value="$(optenv JACKAL_LASER_SECONDARY 0)">
-    <xacro:property name="mount" value="$(optenv JACKAL_LASER_SECONDARY_MOUNT rear)" />
-    <xacro:property name="topic" value="$(optenv JACKAL_LASER_SECONDARY_TOPIC rear/scan)" />
-    <xacro:property name="tower" value="$(optenv JACKAL_LASER_SECONDARY_TOWER 1)" />
-    <xacro:property name="prefix" value="$(optenv JACKAL_LASER_SECONDARY_PREFIX ${mount})" />
-    <xacro:property name="parent" value="$(optenv JACKAL_LASER_SECONDARY_PARENT ${mount}_mount)" />
-    <xacro:property name="lidar_model" value="$(optenv JACKAL_LASER_SECONDARY_MODEL lms1xx)" />
-    <!-- SICK LMS1xx -->
-    <xacro:if value="${lidar_model == 'lms1xx'}">
-      <!-- Mount Enabled -->
-      <xacro:if value="${tower}">
-        <xacro:sick_lms1xx_mount topic="${topic}" prefix="${prefix}" parent_link="${parent}">
-          <origin xyz="$(optenv JACKAL_LASER_SECONDARY_OFFSET 0 0 0)" rpy="$(optenv JACKAL_LASER_SECONDARY_RPY 0 0 3.14159)" />
-        </xacro:sick_lms1xx_mount>
-      </xacro:if>
-      <!-- Mount Disabled -->
-      <xacro:unless value="${tower}">
-        <xacro:sick_lms1xx frame="${prefix}_laser" topic="${topic}" />
-        <link name="${prefix}_laser_base"/>
-        <joint name="${prefix}_laser_base_joint" type="fixed">
-          <origin xyz="$(optenv JACKAL_LASER_SECONDARY_OFFSET 0 0 0)" rpy="$(optenv JACKAL_LASER_SECONDARY_RPY 0 0 3.14159)"/>
-          <parent link="${parent}"/>
-          <child link="${prefix}_laser_base"/>
-        </joint>
-        <joint name="${prefix}_laser_joint" type="fixed">
-          <origin xyz="0 0 0.116" rpy="0 0 0"/>
-          <parent link="${prefix}_laser_base"/>
-          <child link="${prefix}_laser"/>
-        </joint>
-      </xacro:unless>
-    </xacro:if>
-    <!-- SICK Tim -->
-    <xacro:if value="${lidar_model == 'tim551'}">
-      <xacro:property name="prefix" value="$(optenv JACKAL_LASER_SECONDARY_PREFIX tim551_2)" />
-      <xacro:sick_tim551 name="${prefix}" ros_topic="${topic}"/>
-      <joint name="${prefix}_mount_link_joint" type="fixed">
-        <origin xyz="$(optenv JACKAL_LASER_SECONDARY_OFFSET 0 0 0)" rpy="$(optenv JACKAL_LASER_SECONDARY_RPY 0 0 3.14159)"/>
-        <parent link="${parent}"/>
-        <child link="${prefix}_mount_link"/>
-      </joint>
-    </xacro:if>
-    <!-- Hokuyo UST10 -->
-    <xacro:if value="${lidar_model == 'ust10'}">
-      <xacro:hokuyo_ust10_mount topic="${topic}" prefix="${prefix}" parent_link="${parent}">
-        <origin xyz="$(optenv JACKAL_LASER_SECONDARY_OFFSET 0 0 0)" rpy="$(optenv JACKAL_LASER_SECONDARY_RPY 0 0 3.14159)" />
-      </xacro:hokuyo_ust10_mount>
-    </xacro:if>
-    <!-- Hokuyo UTM30 -->
-    <xacro:if value="${lidar_model == 'utm30'}">
-      <xacro:hokuyo_utm30_mount topic="${topic}" prefix="${prefix}" parent_link="${parent}">
-        <origin xyz="$(optenv JACKAL_LASER_SECONDARY_OFFSET 0 0 0)" rpy="$(optenv JACKAL_LASER_SECONDARY_RPY 0 0 3.14159)" />
-      </xacro:hokuyo_utm30_mount>
-    </xacro:if>
-  </xacro:if>
-  <!--
-    Add a 3D lidar sensor.  By default this is a Velodyne VLP16 but can be changed with the
-    JACKAL_LASER_3D_MODEL environment variable. Valid model designations are:
-    - vlp16 (default)  :: Velodyne VLP16
-    - vlp32e           :: Velodyne HDL-32E
-  -->
-  <xacro:if value="$(optenv JACKAL_LASER_3D 0)">
-    <xacro:property name="mount" value="$(optenv JACKAL_LASER_3D_MOUNT mid)" />
-    <xacro:property name="topic" value="$(optenv JACKAL_LASER_3D_TOPIC mid/points)" />
-    <xacro:property name="tower" value="$(optenv JACKAL_LASER_3D_TOWER 1)" />
-    <xacro:property name="prefix" value="$(optenv JACKAL_LASER_3D_PREFIX ${mount})" />
-    <xacro:property name="parent" value="$(optenv JACKAL_LASER_3D_PARENT ${mount}_mount)" />
-    <xacro:property name="lidar_3d_model" value="$(optenv JACKAL_LASER_3D_MODEL vlp16)" />
-    <!-- Velodyne VLP16 -->
-    <xacro:if value="${lidar_3d_model == 'vlp16'}">
-      <xacro:vlp16_mount topic="${topic}" tower="${tower}" prefix="${prefix}" parent_link="${parent}" >
-        <origin xyz="$(optenv JACKAL_LASER_3D_OFFSET 0 0 0)" rpy="$(optenv JACKAL_LASER_3D_RPY 0 0 0)" />
-      </xacro:vlp16_mount>
-    </xacro:if>
-    <!-- Velodyne HDL-32E -->
-    <xacro:if value="${lidar_3d_model == 'hdl32e'}">
-      <xacro:hdl32e_mount topic="${topic}" tower="${tower}" prefix="${prefix}" parent_link="${parent}" >
-        <origin xyz="$(optenv JACKAL_LASER_3D_OFFSET 0 0 0)" rpy="$(optenv JACKAL_LASER_3D_RPY 0 0 0)" />
-      </xacro:hdl32e_mount>
-    </xacro:if>
-  </xacro:if>
-  <!--
-    Add a Nav. Sat. By default this is a Novatel Smart6, but can be changed with the
-    JACKAL_NAVSAT_MODEL environment variable. Valid model designations are:
-    - smart6 (default)    :: Novatel Smart6
-    - smart7              :: Novatel Smart7
-  -->
-  <xacro:include filename="$(find jackal_description)/urdf/accessories/novatel_smart6.urdf.xacro" />
-  <xacro:include filename="$(find jackal_description)/urdf/accessories/novatel_smart7.urdf.xacro" />
-  <xacro:if value="$(optenv JACKAL_NAVSAT 0)">
-    <xacro:property name="mount" value="$(optenv JACKAL_NAVSAT_MOUNT rear)" />
-    <xacro:property name="tower" value="$(optenv JACKAL_NAVSAT_TOWER 1)" />
-    <xacro:property name="prefix" value="$(optenv JACKAL_NAVSAT_PREFIX ${mount})" />
-    <xacro:property name="parent" value="$(optenv JACKAL_NAVSAT_PARENT ${mount}_mount)" />
-    <xacro:property name="navsat_model" value="$(optenv JACKAL_NAVSAT_MODEL smart6)" />
-    <!--- Novotel Smart6 -->
-    <xacro:if value="${navsat_model == 'smart6'}">
-      <xacro:novatel_smart6 prefix="${prefix}"/>
-      <!-- Tower Enabled -->
-      <xacro:if value="${tower}">
-        <xacro:bridge_plate prefix="${prefix}" parent="${parent}" height="$(optenv JACKAL_NAVSAT_HEIGHT 0.1)">
-          <origin xyz="$(optenv JACKAL_NAVSAT_OFFSET 0 0 0)" rpy="$(optenv JACKAL_NAVSAT_RPY 0 0 0)"/>
-        </xacro:bridge_plate>
-        <joint name="${prefix}_navsat_joint" type="fixed">
-          <origin xyz="0 0 0" rpy="0 0 0" />
-          <parent link="${prefix}_bridge" />
-          <child link="${prefix}_navsat" />
-        </joint>
-      </xacro:if>
-      <!-- Tower Disabled -->
-      <xacro:unless value="${tower}">
-        <joint name="${prefix}_navsat_joint" type="fixed">
-          <origin xyz="$(optenv JACKAL_NAVSAT_OFFSET 0 0 0)" rpy="$(optenv JACKAL_NAVSAT_RPY 0 0 0)" />
-          <parent link="${parent}" />
-          <child link="${prefix}_navsat" />
-        </joint>
-      </xacro:unless>
-    </xacro:if>
-    <!-- Novotel Smart7 -->
-    <xacro:if value="${navsat_model == 'smart7'}">
-      <xacro:novatel_smart7 prefix="${prefix}"/>
-      <!-- Tower Enabled -->
-      <xacro:if value="${tower}">
-        <xacro:bridge_plate prefix="${prefix}" parent="${parent}" height="$(optenv JACKAL_NAVSAT_HEIGHT 0.1)">
-          <origin xyz="$(optenv JACKAL_NAVSAT_OFFSET 0 0 0)" rpy="$(optenv JACKAL_NAVSAT_RPY 0 0 0)"/>
-        </xacro:bridge_plate>
-        <joint name="${prefix}_navsat_joint" type="fixed">
-          <origin xyz="0 0 0" rpy="0 0 0" />
-          <parent link="${prefix}_bridge" />
-          <child link="${prefix}_navsat" />
-        </joint>
-      </xacro:if>
-      <!-- Tower Disabled -->
-      <xacro:unless value="${tower}">
-        <joint name="${prefix}_navsat_joint" type="fixed">
-          <origin xyz="$(optenv JACKAL_NAVSAT_OFFSET 0 0 0)" rpy="$(optenv JACKAL_NAVSAT_RPY 0 0 0)" />
-          <parent link="${parent}" />
-          <child link="${prefix}_navsat" />
-        </joint>
-      </xacro:unless>
-    </xacro:if>
-  </xacro:if>
-  <!--
-    Add Cameras.
-    - JACKAL_FLEA3
-    - JACKAL_STEREO_FLEA3
-    - JACKAL_BB2
-  -->
   <!-- Common camera mounts and accessory URDFs. -->
-  <xacro:include filename="$(find jackal_description)/urdf/accessories/camera_mount.urdf.xacro" />
-  <xacro:include filename="$(find pointgrey_camera_description)/urdf/pointgrey_flea3.urdf.xacro" />
+  <!-- <xacro:include filename="$(find jackal_description)/urdf/accessories/camera_mount.urdf.xacro" /> -->
+  <!-- <xacro:include filename="$(find pointgrey_camera_description)/urdf/pointgrey_flea3.urdf.xacro" /> -->
   <!-- If enabled, generate the flea3 camera payload with a tilt of 30 degrees. -->
-  <xacro:if value="$(optenv JACKAL_FLEA3 0)">
-    <xacro:property name="name" value="$(optenv JACKAL_FLEA3_NAME front)" />
-    <xacro:property name="tilt" value="$(optenv JACKAL_FLEA3_TILT 0.5236)" />
-    <xacro:property name="tower" value="$(optenv JACKAL_FLEA3_TOWER 1)" />
-    <xacro:property name="mount" value="$(optenv JACKAL_FLEA3_MOUNT front)" />
-    <xacro:property name="prefix" value="$(optenv JACKAL_FLEA3_PREFIX ${mount})" />
-    <xacro:property name="parent" value="$(optenv JACKAL_FLEA3_PARENT ${mount}_mount)" />
-    <xacro:pointgrey_flea3 frame="${prefix}_camera" name="${name}"
+  <!-- <xacro:if value="$(optenv JACKAL_FLEA3 0)">
+    <camera_mount prefix="$(optenv JACKAL_FLEA3_MOUNT front)"
+                       tilt="$(optenv JACKAL_FLEA3_TILT 0.5236)"/>
+    <joint name="$(optenv JACKAL_FLEA3_MOUNT front)_camera_mount_joint" type="fixed">
+      <origin xyz="$(optenv JACKAL_FLEA3_OFFSET 0 0 0)"
+              rpy="$(optenv JACKAL_FLEA3_RPY 0 0 0)" />
+      <parent link="$(optenv JACKAL_FLEA3_MOUNT front)_mount" />
+      <child link="$(optenv JACKAL_FLEA3_MOUNT front)_camera_mount" />
+    </joint>
+    <pointgrey_flea3 frame="$(optenv JACKAL_FLEA3_MOUNT front)_camera" name="$(optenv JACKAL_FLEA3_NAME front)"
       camera_x="0.0754" camera_y="0.029" camera_z="0.029"
       camera_mass="0.085" hfov="1.0471975512" fps="60" width="640" height="512"/>
-    <!-- Mount Enabled -->
-    <xacro:if value="${tower}">
-      <xacro:camera_mount prefix="${prefix}" tilt="${tilt}"/>
-      <joint name="${prefix}_camera_mount_joint" type="fixed">
-        <origin xyz="$(optenv JACKAL_FLEA3_OFFSET 0 0 0)"
-                rpy="$(optenv JACKAL_FLEA3_RPY 0 0 0)" />
-        <parent link="${parent}" />
-        <child link="${prefix}_camera_mount" />
-      </joint>
-      <joint name="${prefix}_camera_bracket_joint" type="fixed">
-        <origin xyz="0.020 0 0.0245" rpy="0 0 0" />
-        <parent link="${prefix}_camera_beam" />
-        <child link="${prefix}_camera" />
-      </joint>
-    </xacro:if>
-    <!-- Mount Disabled -->
-    <xacro:unless value="${tower}">
-      <link name="${prefix}_camera_base"/>
-      <joint name="${prefix}_camera_base_joint" type="fixed">
-        <origin xyz="$(optenv JACKAL_FLEA3_OFFSET 0 0 0)"
-                rpy="$(optenv JACKAL_FLEA3_RPY 0 0 0)" />
-        <parent link="${parent}" />
-        <child link="${prefix}_camera_base" />
-      </joint>
-      <joint name="${prefix}_camera_joint" type="fixed">
-        <origin xyz="0 0 0.0145"
-                rpy="0 0 0" />
-        <parent link="${prefix}_camera_base" />
-        <child link="${prefix}_camera" />
-      </joint>
-    </xacro:unless>
-  </xacro:if>
-  <xacro:include filename="$(find jackal_description)/urdf/accessories/stereo_camera_mount.urdf.xacro" />
+    <joint name="$(optenv JACKAL_FLEA3_MOUNT front)_camera_bracket_joint" type="fixed">
+      <origin xyz="0.020 0 0.0245" rpy="0 0 0" />
+      <parent link="$(optenv JACKAL_FLEA3_MOUNT front)_camera_beam" />
+      <child link="$(optenv JACKAL_FLEA3_MOUNT front)_camera" />
+    </joint>
+  </xacro:if> -->
+  <!-- <xacro:include filename="$(find jackal_description)/urdf/accessories/stereo_camera_mount.urdf.xacro" /> -->
   <!-- If enabled, generates a pair of flea3 cameras for stereo vision with a tilt of 30 degrees. -->
   <!-- Disabled temporarily due to metapackage issue. -->
-  <xacro:if value="$(optenv JACKAL_STEREO_FLEA3 0)">
-    <xacro:property name="tilt" value="$(optenv JACKAL_FLEA3_TILT 0.5236)"/>
-    <xacro:property name="mount" value="$(optenv JACKAL_FLEA3_MOUNT front)"/>
-    <xacro:property name="prefix" value="$(optenv JACKAL_FLEA3_PREFIX ${mount})"/>
-    <xacro:property name="parent" value="$(optenv JACKAL_FLEA3_PARENT ${mount}_mount)"/>
-    <xacro:property name="left_name" value="$(optenv JACKAL_FLEA3_LEFT_NAME front/left)"/>
-    <xacro:property name="right_name" value="$(optenv JACKAL_FLEA3_RIGHT_NAME front/right)"/>
-    <xacro:property name="separation" value="$(optenv JACKAL_STEREO_SEPERATION 0.16)"/>
-    <xacro:stereo_camera_mount prefix="${prefix}" tilt="${tilt}"/>
-    <joint name="${prefix}_stereo_camera_mount_joint" type="fixed">
+  <!-- <xacro:if value="$(optenv JACKAL_STEREO_FLEA3 0)">
+    <stereo_camera_mount prefix="$(optenv JACKAL_FLEA3_MOUNT front)"
+                       tilt="$(optenv JACKAL_FLEA3_TILT 0.5236)"/>
+    <joint name="$(optenv JACKAL_FLEA3_MOUNT front)_stereo_camera_mount_joint" type="fixed">
       <origin xyz="$(optenv JACKAL_FLEA3_OFFSET 0 0 0)"
               rpy="$(optenv JACKAL_FLEA3_RPY 0 0 0)" />
-      <parent link="${parent}" />
-      <child link="${prefix}_stereo_camera_mount" />
+      <parent link="$(optenv JACKAL_FLEA3_MOUNT front)_mount" />
+      <child link="$(optenv JACKAL_FLEA3_MOUNT front)_stereo_camera_mount" />
     </joint>
-    <xacro:pointgrey_flea3 frame="${prefix}_left_camera" name="${left_name}"
+    <pointgrey_flea3 frame="$(optenv JACKAL_FLEA3_MOUNT front)_left_camera" name="$(optenv JACKAL_FLEA3_LEFT_NAME front/left)"
       camera_x="0.0754" camera_y="0.029" camera_z="0.029"
       camera_mass="0.085" hfov="1.0471975512" fps="60" width="640" height="512"/>
-    <joint name="${prefix}_left_stereo_camera_bracket_joint" type="fixed">
-      <origin xyz="0.015 ${separation} 0.0599" rpy="0 0 0" />
-      <parent link="${prefix}_stereo_camera_beam" />
-      <child link="${prefix}_left_camera" />
+    <joint name="$(optenv JACKAL_FLEA3_MOUNT front)_left_stereo_camera_bracket_joint" type="fixed">
+      <origin xyz="0.015 $(optenv JACKAL_STEREO_SEPERATION 0.16) 0.0599" rpy="0 0 0" />
+      <parent link="$(optenv JACKAL_FLEA3_MOUNT front)_stereo_camera_beam" />
+      <child link="$(optenv JACKAL_FLEA3_MOUNT front)_left_camera" />
     </joint>
-    <xacro:pointgrey_flea3 frame="${prefix}_right_camera" name="${right_name}"
+    <pointgrey_flea3 frame="$(optenv JACKAL_FLEA3_MOUNT front)_right_camera" name="$(optenv JACKAL_FLEA3_RIGHT_NAME front/right)"
       camera_x="0.0754" camera_y="0.029" camera_z="0.029"
       camera_mass="0.085" hfov="1.0471975512" fps="60" width="640" height="512"/>
-    <joint name="${prefix}_right_stereo_camera_bracket_joint" type="fixed">
-      <origin xyz="0.015 -${separation} 0.0599" rpy="0 0 0" />
-      <parent link="${prefix}_stereo_camera_beam" />
-      <child link="${prefix}_right_camera" />
+    <joint name="$(optenv JACKAL_FLEA3_MOUNT front)_right_stereo_camera_bracket_joint" type="fixed">
+      <origin xyz="0.015 -$(optenv JACKAL_STEREO_SEPERATION 0.16) 0.0599" rpy="0 0 0" />
+      <parent link="$(optenv JACKAL_FLEA3_MOUNT front)_stereo_camera_beam" />
+      <child link="$(optenv JACKAL_FLEA3_MOUNT front)_right_camera" />
     </joint>
-  </xacro:if>
+  </xacro:if> -->
   <!-- If enabled, generate the bumblebee2 camera payload with a tilt of 0 degrees. -->
-  <xacro:include filename="$(find pointgrey_camera_description)/urdf/pointgrey_bumblebee2.urdf.xacro" />
+  <!-- <xacro:include filename="$(find pointgrey_camera_description)/urdf/pointgrey_bumblebee2.urdf.xacro" /> -->
   <!-- If enabled, generate the bumblebee2 camera payload with a tilt of 0 degrees. -->
   <!-- Disabled temporarily due to metapackage issue. -->
-  <xacro:if value="$(optenv JACKAL_BB2 0)">
-    <xacro:property name="tilt" value="$(optenv JACKAL_BB2_TILT 0)" />
-    <xacro:property name="name" value="$(optenv JACKAL_BB2_NAME front)" />
-    <xacro:property name="tower" value="$(optenv JACKAL_BB2_TOWER 1)"/>
-    <xacro:property name="mount" value="$(optenv JACKAL_BB2_MOUNT front)" />
-    <xacro:property name="prefix" value="$(optenv JACKAL_BB2_PREFIX ${mount})"/>
-    <xacro:property name="parent" value="$(optenv JACKAL_BB2_PARENT ${mount}_mount)"/>
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