Commit message: article publish

File: jackal_description/urdf/accessories/bridge_plate.urdf.xacro (robot description, xacro)
@@ -1,17 +1,11 @@
 <?xml version="1.0"?>
 <robot xmlns:xacro="http://www.ros.org/wiki/xacro">
-  <xacro:macro name="bridge_plate" params="prefix parent height *origin">
-    <link name="${prefix}_bridge_base"/>
-    <joint name="${prefix}_bridge_base_joint" type="fixed">
-      <parent link="${parent}"/>
-      <child link="${prefix}_bridge_base" />
-      <xacro:insert_block name="origin" />
-    </joint>
-    <joint name="${prefix}_bridge_joint" type="fixed">
-      <parent link="${prefix}_bridge_base"/>
-      <child link="${prefix}_bridge"/>
+  <xacro:macro name="bridge_plate" params="mount height">
+    <joint name="${mount}_mount_to_${mount}_bridge" type="fixed">
+      <parent link="${mount}_mount"/>
+      <child link="${mount}_bridge"/>
       <origin xyz="0.0 0.0 ${height}" rpy="0 0 0"/>
     </joint>
-    <link name="${prefix}_bridge">
+    <link name="${mount}_bridge">
       <visual>
         <origin xyz="0 0 0" rpy="1.5707 0.0 1.5707" />
@@ -22,5 +16,5 @@
       </visual>
     </link>
-    <xacro:standoff_box prefix="${prefix}" parent="${prefix}_bridge_base" height="${height}" />
+    <standoff_box mount="${mount}" height="${height}" />
   </xacro:macro>
 </robot>

File: jackal_description/urdf/accessories/hokuyo_ust10.urdf.xacro (robot description, xacro)
@@ -1,5 +1,5 @@
 <?xml version="1.0"?>
 <robot xmlns:xacro="http://ros.org/wiki/xacro">
-  <xacro:macro name="hokuyo_ust10_mount" params="prefix topic parent_link min_angle:=-2.35619 max_angle:=2.35619 *origin">
+  <xacro:macro name="hokuyo_ust10_mount" params="prefix topic parent_link">
     <xacro:macro name="hokuyo_ust10" params="frame:=laser topic:=scan sample_size:=720 update_rate:=50
                min_angle:=-2.35619 max_angle:=2.35619 min_range:=0.1 max_range:=30.0 robot_namespace:=/">
@@ -47,7 +47,8 @@
       </gazebo>
     </xacro:macro>
-    <xacro:hokuyo_ust10 frame="${prefix}_laser" topic="${topic}"/>
+    <hokuyo_ust10 frame="${prefix}_laser" topic="${topic}"/>
     <joint name="${prefix}_laser_mount_joint" type="fixed">
-      <xacro:insert_block name="origin" />
+      <origin xyz="$(optenv JACKAL_LASER_OFFSET 0 0 0)"
+              rpy="$(optenv JACKAL_LASER_RPY 0 0 0)" />
       <parent link="${parent_link}" />
       <child link="${prefix}_laser_mount" />

File: jackal_description/urdf/accessories/standoffs.urdf.xacro (robot description, xacro)
@@ -19,17 +19,17 @@
   </xacro:macro>
   <!-- Generate a set of four standoffs from a payload mount point. -->
-  <xacro:macro name="standoff_box" params="prefix parent height">
-    <xacro:standoff name="${prefix}_standoff0" length="${height}" parent="${parent}">
+  <xacro:macro name="standoff_box" params="mount height">
+    <standoff name="${mount}_standoff0" length="${height}" parent="${mount}_mount">
       <origin xyz="0.060 0.060 0" rpy="0 0 0"/>
-    </xacro:standoff>
-    <xacro:standoff name="${prefix}_standoff1" length="${height}" parent="${parent}">
+    </standoff>
+    <standoff name="${mount}_standoff1" length="${height}" parent="${mount}_mount">
       <origin xyz="0.060 -0.060 0" rpy="0 0 0"/>
-    </xacro:standoff>
-    <xacro:standoff name="${prefix}_standoff2" length="${height}" parent="${parent}">
+    </standoff>
+    <standoff name="${mount}_standoff2" length="${height}" parent="${mount}_mount">
       <origin xyz="-0.060 0.060 0" rpy="0 0 0"/>
-    </xacro:standoff>
-    <xacro:standoff name="${prefix}_standoff3" length="${height}" parent="${parent}">
+    </standoff>
+    <standoff name="${mount}_standoff3" length="${height}" parent="${mount}_mount">
       <origin xyz="-0.060 -0.060 0" rpy="0 0 0"/>
-    </xacro:standoff>
+    </standoff>
   </xacro:macro>
 </robot>

File: jackal_description/urdf/jackal.urdf.xacro (robot description, xacro)
@@ -173,5 +173,8 @@
     <child link="rear_fender_link" />
   </joint>
-  <!-- Default Internal IMU Link -->
+  <!-- TODO: Make this internal_imu_link or something, and use a mixed-in xacro
+       to supply the joint between it and imu_link. This is important so that imu_link
+       always points to the "active" IMU. When an upgrade IMU is connected, the
+       internal_imu_link should remain, but imu_link should point to the upgrade one. -->
   <link name="imu_link">
     <inertial>
@@ -185,5 +188,5 @@
     <child link="imu_link" />
   </joint>
-  <!-- Default NAVSAT Link -->
+  <!-- TODO: Same note as applies to imu_link -->
   <link name="navsat_link">
     <visual>
@@ -224,15 +227,5 @@
        default each one to off.-->
   <xacro:include filename="$(find jackal_description)/urdf/accessories.urdf.xacro" />
-  <!-- OutdoorNav -->
-  <xacro:arg name="outdoornav_enabled"       default="$(optenv OUTDOORNAV_ENABLED 0)" />
-  <xacro:arg name="outdoornav_configuration" default="$(optenv OUTDOORNAV_CONFIGURATION standard)" />
-  <!-- OutdoorNav URDF Config -->
-  <xacro:if value="$(arg outdoornav_enabled)">
-    <xacro:include filename="$(find cpr_onav_description)/urdf/outdoornav_description.urdf.xacro" />
-    <xacro:outdoornav_sensors outdoornav_configuration="$(arg outdoornav_configuration)" />
-  </xacro:if>
   <!-- Optional custom includes. -->
   <xacro:include filename="$(optenv JACKAL_URDF_EXTRAS empty.urdf)" />
-  <!-- Optional for Clearpath internal softwares -->
-  <xacro:include filename="$(optenv CPR_URDF_EXTRAS empty.urdf)" />
 </robot>
